File: Hardware/simpleSBC.kicad_pcb (KiCad board)
At the start: 6 copper layers, 66 x 56 mm, 192 parts, among them J1 Conn_02x07_Odd_Even, J2 Micro_SD_Card_Det2, J4 Barrel_Jack_Switch, J5 USB_A, J6 USB_A, J7 RJ45_Wuerth_7499010121A, J8 Conn_01x03, J9 Conn_01x06, U1 STM32MP157FAD1, U2 STMPS2252MTR, U3 MT41K256M16TW, U4 STPMIC1, U5 USBLC6-4SC6, U6 LAN8742A, X1 ASCO, Y1 32.786

Commit message: First Pass Routing
Parts:
- removed R59, R9: 0, Resistor_SMD:R_0402_1005Metric
- added C98: 22u, Capacitor_SMD:C_0805_2012Metric, F.Cu at (133.8, 97.0)
- added C99: 4.7u, Capacitor_SMD:C_0402_1005Metric, F.Cu at (134.2, 99.0)
- added JP2: SolderJumper_2_Bridged, Resistor_SMD:R_0402_1005Metric, F.Cu at (113.0, 90.0)
- added JP3: SolderJumper_2_Bridged, Resistor_SMD:R_0402_1005Metric, F.Cu at (114.0, 90.0)
- added JP4: SolderJumper_3_Bridged12, Jumper:SolderJumper-3_P1.3mm_Bridged2Bar12_Pad1.0x1.5mm, B.Cu at (134.0, 98.8)
- added JP5: SolderJumper_3_Bridged12, Jumper:SolderJumper-3_P1.3mm_Bridged2Bar12_Pad1.0x1.5mm, B.Cu at (121.2, 99.5)
- added JP6: SolderJumper_3_Bridged12, Jumper:SolderJumper-3_P1.3mm_Bridged2Bar12_Pad1.0x1.5mm, B.Cu at (125.0, 72.8)
- added JP7: SolderJumper_3_Bridged12, Jumper:SolderJumper-3_P1.3mm_Bridged2Bar12_Pad1.0x1.5mm, B.Cu at (144.4, 72.8)
- added L5: 1u, Inductor_SMD:L_1008_2520Metric, F.Cu at (137.0, 98.8)
- added SW1: SW_Push, Button_Switch_SMD:SW_SPST_Omron_B3FS-101xP, F.Cu at (161.8, 106.5)
- added Y3: 24M, SimpleSBC:Crystal_2.00x1.60mm, F.Cu at (155.5, 72.4)
- JP1: footprint Jumper:SolderJumper-2_P1.3mm_Bridged2Bar_Pad1.0x1.5mm -> Resistor_SMD:R_0402_1005Metric
- R48, TP8: moved to B.Cu
- moved J9 33.0 mm to (204.2, 92.8)
- moved TP1 28.8 mm to (127.4, 100.7)
- moved R48 23.2 mm to (148.9, 79.0), turned to 90 degrees
- moved R47 22.7 mm to (151.3, 77.2), turned to 90 degrees
- moved R44 22.3 mm to (150.5, 74.8), turned to 0 degrees
- moved C42 22.3 mm to (154.9, 70.2), turned to 90 degrees
- moved R40 22.1 mm to (159.0, 61.2), turned to 0 degrees
- moved C79 22.1 mm to (153.4, 72.3), turned to 180 degrees
- moved C43 21.5 mm to (152.3, 76.8), turned to -90 degrees
- moved C80 21.4 mm to (153.4, 73.3), turned to 180 degrees
- moved JP1 20.6 mm to (148.5, 96.6)
- moved R49 20.5 mm to (152.0, 74.2)
- moved C44 20.3 mm to (157.0, 70.2), turned to 90 degrees
- moved R43 20.1 mm to (149.8, 77.0), turned to 0 degrees
- moved D1 19.5 mm to (159.6, 62.8), turned to 180 degrees
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Connections:
- net Net-(J5-D+) renamed /USB2_D+
- net Net-(J5-D-) renamed /USB2_D-
- net Net-(J6-D+) renamed /USB1_D-
- net Net-(J6-D-) renamed /USB1_D+
- C39 pad 2: +5V -> VBUS
- C41 pad 2: +5V -> VBUS
- FB1 pad 1: +5V -> VBUS
- JP1 pad 1: Net-(JP1-A) -> /Power/~{RST}
- JP1 pad 2: +3V3 -> /NRST
- R10 pad 2: +3V3 -> +3.3VP
- R11 pad 2: +3V3 -> +3.3VP
- R12 pad 2: +3V3 -> +3.3VP
- R13 pad 2: +3V3 -> +3.3VP
- R14 pad 2: +3V3 -> +3.3VP
- R15 pad 2: +3V3 -> +3.3VP
- U1 pad V7: unconnected-(U1B-PE7-PadV7) -> /USB_~{OC2}
- U1 pad V9: unconnected-(U1B-PF9-PadV9) -> /USB_~{OC1}
- U1 pad W7: /IO5 -> /PRT1
- U1 pad W8: /IO6 -> /PRT2
- U2 pad 6: Net-(J5-VBUS) -> /VBUS2
- U2 pad 7: Net-(J6-VBUS) -> /VBUS1
- U4 pad 34: unconnected-(U4-BSTOUT-Pad34) -> /Power/VOUT_BST
- U4 pad 35: unconnected-(U4-VBUSOTG-Pad35) -> /PMIC_VBUSOTG
- U4 pad 38: unconnected-(U4-SWOUT-Pad38) -> /PMIC_SWOUT
Routing:
- net GND: track 76.0 -> 137.2 mm, vias 56 -> 70
- net Net-(JP3-A): track 0.00 -> 58.6 mm, vias 0 -> 2
- net /PMIC_SWOUT: track 0.00 -> 56.2 mm, vias 0 -> 3
- net Net-(JP2-A): track 0.00 -> 56.1 mm, vias 0 -> 2
- net /PA0_WAKEUP: track 0.00 -> 40.1 mm, vias 0 -> 3
- net /PRT1: track 0.00 -> 39.6 mm, vias 0 -> 2
- net /PRT2: track 0.00 -> 39.5 mm, vias 0 -> 2
- net /USB_~{OC2}: track 0.00 -> 38.4 mm, vias 0 -> 2
- net /ETH_TX-: track 0.00 -> 37.5 mm
- net /NRST: track 5.71 -> 43.2 mm, vias 2 -> 3
- net +3V3: track 20.0 -> 56.6 mm, vias 10 -> 31
- net VDD_USB: track 0.00 -> 36.4 mm, vias 0 -> 4
- net /SDMMC_D0: track 3.34 -> 39.4 mm, vias 1 -> 2
- net /ETH_TX+: track 0.00 -> 35.3 mm
- net /SDMMC_D1: track 4.03 -> 39.3 mm, vias 1 -> 2
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- added copper zone on F.Cu, net +1V2
- added copper zone on F.Cu, net +1V35
- added copper zone on F.Cu, net +3.3VP
- added copper zone on F.Cu, net +3V3
- added copper zone on F.Cu, net +5V
- added copper zone on In4.Cu, net +5V
- added copper zone on F.Cu, net /Power/VOUT_BST
- added copper zone on F.Cu, net Net-(U4-VLX1)
- added copper zone on F.Cu, net Net-(U4-VLX2)
- added copper zone on F.Cu, net Net-(U4-VLX3)
- added copper zone on F.Cu, net Net-(U4-VLX4)
- added copper zone on F.Cu, net Net-(U4-VLXBST)
Other:
- board size 66 x 56 mm -> 82.7 x 56 mm
- board text added: "VDD_USB?"
