File: Hardware/power.kicad_sch (KiCad schematic)
At the start: 80 parts, among them J4 Barrel_Jack_Switch, J8 Conn_01x03, U1 STM32MP157FAD1, U4 STPMIC1A

Commit message: prepare for assembly
Parts:
- C1, C11, C13, C15, C18, C21, C23, C24, C26, C28, C3, C30, C31, C32, C35, C38, C48, C5, C67, C68, C7, C75: JLCPCB Part # (none) -> C52923
- C10, C17: JLCPCB Part # (none) -> C1523
- C12, C14, C16, C19, C20, C22, C25, C27, C4, C46, C49, C6, C8, C9: JLCPCB Part # (none) -> C1525
- C33, C34: JLCPCB Part # (none) -> C15850
- C69, C74, C76, C86, C88, C95, C96, C99: JLCPCB Part # (none) -> C23733
- C70, C71, C72, C73, C87, C89, C94: JLCPCB Part # (none) -> C19702
- C90, C91, C92, C93, C98: JLCPCB Part # (none) -> C45783
- J4, J8, JP5, TP1, TP10, TP2, TP3, TP4, TP5, TP6: now not fitted
- L1, L2, L3, L4, L5: JLCPCB Part # (none) -> C76795
- R57, R58: JLCPCB Part # (none) -> C25879
- U1: JLCPCB Part # (none) -> C1236719
- U4: JLCPCB Part # (none) -> C2156050
