File: Hardware/simpleSBC.kicad_sch (KiCad schematic)
At the start: 72 parts, among them J1 Conn_02x07_Odd_Even, J3 Conn_02x10_Odd_Even, J5 USB_A, J6 USB_A, J7 RJ45_Wuerth_7499010121A, J9 Conn_02x10_Odd_Even, SW1 SW_Push, U1 STM32MP157FAD1, U2 STMPS2252MTR, U5 USBLC6-4SC6, U6 LAN8742A, X1 ASCO, Y1 32.786, Y3 24M

Commit message: Stale changes
Parts:
- Y3: value 24M -> 25M
Changed lines of the file:
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@@
 			)
 		)
-		(property "Value" "24M"
+		(property "Value" "25M"
 			(at 94.234 176.784 90)
 			(effects
